File: rev1/pcb/pakbd/pakbd.sch (KiCad schematic (older format))
At the start: 158 parts, among them J0 MJ-4PP-9, J1 MJ-4PP-9, SW0 SW_Push, SW1 SW_Push, SW10 SW_Push, SW11 SW_Push, SW12 SW_Push, SW13 SW_Push, SW14 SW_Push, SW15 SW_Push, SW16 SW_Push, SW17 SW_Push, SW18 SW_Push, SW19 SW_Push, SW2 SW_Push, SW20 SW_Push, SW21 SW_Push, SW22 SW_Push, SW23 SW_Push, SW24 SW_Push, SW25 SW_Push, SW26 SW_Push, SW27 SW_Push, SW28 SW_Push, SW29 SW_Push, SW3 SW_Push, SW30 SW_Push, SW31 SW_Push, SW32 SW_Push, SW33 SW_Push, SW34 SW_Push, SW35 SW_Push, SW36 SW_Push, SW37 SW_Push, SW38 SW_Push, SW39 SW_Push, SW4 SW_Push, SW40 SW_Push, SW41 SW_Push, SW42 SW_Push, SW43 SW_Push, SW44 SW_Push, SW45 SW_Push, SW46 SW_Push, SW47 SW_Push, SW48 SW_Push, SW49 SW_Push, SW5 SW_Push, SW50 SW_Push, SW51 SW_Push, SW52 SW_Push, SW53 SW_Push, SW54 SW_Push, SW55 SW_Push, SW56 SW_Push, SW57 SW_Push, SW58 SW_Push, SW59 SW_Push, SW6 SW_Push, SW60 SW_Push, SW61 SW_Push, SW62 SW_Push, SW63 SW_Push, SW64 SW_Push, SW65 SW_Push, SW66 SW_Push, SW67 SW_Push, SW68 SW_Push, SW69 SW_Push, SW7 SW_Push, SW8 SW_Push, SW9 SW_Push, U0 ProMicro, U1 ProMicro

Commit message: Add footprint
Parts:
- D0, D1, D10, D11, D12, D13, D14, D15, D16, D17, D18, D19, D2, D20, D21, D22, D23, D24, D25, D26, D27, D28, D29, D3, D30, D31, D32, D33, D34, D35, D36, D37, D38, D39, D4, D40, D41, D42, D43, D44, D45, D46, D47, D48, D49, D5, D50, D51, D52, D53, D54, D55, D56, D57, D58, D59, D6, D60, D61, D62, D63, D64, D65, D66, D67, D68, D69, D7, D8, D9: footprint (none) -> Diode_SMD:D_1206_3216Metric_Pad1.42x1.75mm_HandSolder
- J0, J1: footprint (none) -> MJ-4PP-9:MJ-4PP-9
- JP_da0, JP_da1, JP_db0, JP_db1, JP_xa0, JP_xa1, JP_xb0, JP_xb1: footprint (none) -> Jumper:SolderJumper-2_P1.3mm_Open_Pad1.0x1.5mm
- R_data0, R_data1, R_xdata0, R_xdata1: footprint (none) -> Resistor_SMD:R_1206_3216Metric_Pad1.42x1.75mm_HandSolder
- SW0, SW1, SW10, SW11, SW12, SW13, SW15, SW16, SW17, SW18, SW19, SW2, SW20, SW22, SW23, SW24, SW25, SW26, SW29, SW3, SW30, SW31, SW32, SW33, SW34, SW35, SW36, SW37, SW38, SW39, SW4, SW40, SW41, SW42, SW43, SW44, SW45, SW46, SW47, SW48, SW49, SW5, SW50, SW51, SW52, SW53, SW55, SW56, SW57, SW58, SW59, SW6, SW60, SW61, SW63, SW64, SW67, SW68, SW69, SW8, SW9: footprint (none) -> CPG151101S11:CPG151101S11_1.00u_PCB
- SW14, SW21, SW54: footprint (none) -> CPG151101S11:CPG151101S11_1.75u_PCB
- SW27, SW28, SW62, SW65, SW66: footprint (none) -> CPG151101S11:CPG151101S11_1.25u_PCB
- SW7: footprint (none) -> CPG151101S11:CPG151101S11_1.50u_PCB
- SW_r0, SW_r1: footprint (none) -> Button_Switch_THT:SW_Tactile_Straight_KSA0Axx1LFTR
- U0, U1: footprint (none) -> promicro:ProMicro
