File: rev1/pcb/pakbd/pakbd.kicad_pcb (KiCad board)
At the start: 2 copper layers, 368.3 x 99.3 mm, 190 parts, among them J0 MJ-4PP-9, J1 MJ-4PP-9, SW0 SW_Push, SW1 SW_Push, SW10 SW_Push, SW11 SW_Push, SW12 SW_Push, SW13 SW_Push, SW14 SW_Push, SW15 SW_Push, SW16 SW_Push, SW17 SW_Push, SW18 SW_Push, SW19 SW_Push, SW2 SW_Push, SW20 SW_Push, SW21 SW_Push, SW22 SW_Push, SW23 SW_Push, SW24 SW_Push, SW25 SW_Push, SW26 SW_Push, SW27 SW_Push, SW28 SW_Push, SW29 SW_Push, SW3 SW_Push, SW30 SW_Push, SW31 SW_Push, SW32 SW_Push, SW33 SW_Push, SW34 SW_Push, SW35 SW_Push, SW36 SW_Push, SW37 SW_Push, SW38 SW_Push, SW39 SW_Push, SW4 SW_Push, SW40 SW_Push, SW41 SW_Push, SW42 SW_Push, SW43 SW_Push, SW44 SW_Push, SW45 SW_Push, SW46 SW_Push, SW47 SW_Push, SW48 SW_Push, SW49 SW_Push, SW5 SW_Push, SW50 SW_Push, SW51 SW_Push, SW52 SW_Push, SW53 SW_Push, SW54 SW_Push, SW55 SW_Push, SW56 SW_Push, SW57 SW_Push, SW58 SW_Push, SW59 SW_Push, SW6 SW_Push, SW60 SW_Push, SW61 SW_Push, SW62 SW_Push, SW63 SW_Push, SW64 SW_Push, SW65 SW_Push, SW66 SW_Push, SW67 SW_Push, SW68 SW_Push, SW69 SW_Push, SW7 SW_Push, SW8 SW_Push, SW9 SW_Push, U0 ProMicro, U1 ProMicro

Commit message: Add wiring
Parts:
- moved JP_db1 43.6 mm to (340.1, 81.4), turned to 180 degrees
- moved JP_xa0 42.5 mm to (28.4, 113.7), turned to 270 degrees
- moved JP_da1 42.1 mm to (340.1, 77.8), turned to 180 degrees
- moved R_data1 40.3 mm to (340.9, 75.1), turned to 180 degrees
- moved R_xdata0 37.2 mm to (34.4, 118.6)
- moved JP_xb0 33.2 mm to (38.5, 113.7), turned to 270 degrees
- moved JP_da0 32.2 mm to (30.9, 113.7), turned to 270 degrees
- moved R_data0 30.9 mm to (34.4, 122.5)
- moved JP_xb1 30.4 mm to (340.1, 92.6), turned to 180 degrees
- moved JP_xa1 28.8 mm to (340.1, 89.0), turned to 180 degrees
- moved R_xdata1 27.3 mm to (340.9, 85.8), turned to 180 degrees
- moved JP_db0 23.2 mm to (41.2, 113.7), turned to 270 degrees
- moved h00 1.00 mm to (25.9, 32.9)
- moved h01 1.00 mm to (156.7, 32.9)
- moved h06 1.00 mm to (25.9, 129.6)
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Routing:
- net col7: track 0.00 -> 288.6 mm, vias 0 -> 1
- net row9: track 0.00 -> 248.2 mm, vias 0 -> 1
- net col8: track 0.00 -> 246.4 mm, vias 0 -> 9
- net col3: track 0.00 -> 221.1 mm, vias 0 -> 8
- net col9: track 0.00 -> 220.7 mm, vias 0 -> 9
- net col10: track 0.00 -> 198.8 mm, vias 0 -> 9
- net row5: track 0.00 -> 197.3 mm, vias 0 -> 1
- net row6: track 0.00 -> 188.7 mm, vias 0 -> 1
- net col5: track 0.00 -> 186.8 mm, vias 0 -> 6
- net row0: track 0.00 -> 184.4 mm, vias 0 -> 1
- net col2: track 0.00 -> 180.5 mm, vias 0 -> 8
- net col4: track 0.00 -> 179.2 mm, vias 0 -> 6
- net col11: track 0.00 -> 179.0 mm, vias 0 -> 9
- net VCC: track 0.00 -> 170.1 mm, vias 0 -> 4
- net row1: track 0.00 -> 169.0 mm, vias 0 -> 1
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- added copper zone on B.Cu, net (none)
- added copper zone on F.Cu, net (none)
Other:
- board size 368.3 x 99.3 mm -> 368.3 x 101.3 mm
- board text added: "@yskoht"
- board text added: "pakbd rev1"
